File: Li-po_chargers_tester.kicad_sch (KiCad schematic)
At the start: 42 parts, among them J1 Conn_01x04_Pin, J2 USB_C_Receptacle_PowerOnly_6P, SW1 SW_DIP_x04, U1 BQ24073RGT, U2 MCP73831-3-OT, U3 MCP73833-xxx-MF

Commit message: Board making #1 I made the whole PCB board. Just minor bug repairment and then it should be good
Parts:
- added GND1: GND, TestPoint:TestPoint_Pad_D1.5mm, symbol Connector:TestPoint
- renumbered J1 to STAT3
Connections:
- net GND: now also GND1.1
- net at R8.2, U3.7 (~{PG}): now also STAT2.1 (Pin_1); no longer STAT2.3 (Pin_3)
- net at R6.2, U3.3 (STAT1): now also STAT2.3 (Pin_3); no longer STAT2.1 (Pin_1)
Other:
- note added: "1.8$"
- note removed: "0.95$"
- moved on the sheet: STAT2
Changed lines of the file:
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@@
 	)
 	(junction
+		(at 59.69 185.42)
+		(diameter 0)
+		(color 0 0 0 0)
+	)
+	(junction
 		(at 60.96 171.45)
 		(diameter 0)
@@
 	(wire
 		(pts
+			(xy 106.68 93.98) (xy 106.68 97.79)
+		)
+		(stroke
+			(width 0)
+			(type default)
+		)
+	)
+	(wire
+		(pts
 			(xy 81.28 182.88) (xy 83.82 182.88)
 		)
@@
 	(wire
 		(pts
+			(xy 113.03 97.79) (xy 115.57 97.79)
+		)
+		(stroke
+			(width 0)
+			(type default)
+		)
+	)
+	(wire
+		(pts
 			(xy 60.96 168.91) (xy 60.96 171.45)
 		)
@@
 	(wire
 		(pts
+			(xy 114.3 100.33) (xy 114.3 101.6)
+		)
+		(stroke
+			(width 0)
+			(type default)
+		)
+	)
+	(wire
+		(pts
 			(xy 214.63 105.41) (xy 219.71 105.41)
 		)
@@
 	(wire
 		(pts
+			(xy 59.69 185.42) (xy 50.8 185.42)
+		)
+		(stroke
+			(width 0)
+			(type default)
+		)
+	)
+	(wire
+		(pts
 			(xy 139.7 97.79) (xy 140.97 97.79)
 		)
@@
 	(wire
 		(pts
+			(xy 106.68 105.41) (xy 106.68 102.87)
+		)
+		(stroke
+			(width 0)
+			(type default)
+		)
+	)
+	(wire
+		(pts
 			(xy 245.11 107.95) (xy 245.11 119.38)
 		)
@@
 	(wire
 		(pts
+			(xy 113.03 93.98) (xy 106.68 93.98)
+		)
+		(stroke
+			(width 0)
+			(type default)
+		)
+	)
+	(wire
+		(pts
 			(xy 218.44 63.5) (xy 220.98 63.5)
 		)
@@
 	(wire
 		(pts
-			(xy 60.96 185.42) (xy 50.8 185.42)
+			(xy 60.96 185.42) (xy 59.69 185.42)
 		)
 		(stroke
@@
 	(wire
 		(pts
-			(xy 115.57 97.79) (xy 114.3 97.79)
-		)
-		(stroke
-			(width 0)
-			(type default)
-		)
-	)
-	(wire
-		(pts
 			(xy 232.41 114.3) (xy 232.41 113.03)
 		)
@@
 	(wire
 		(pts
+			(xy 106.68 101.6) (xy 106.68 100.33)
+		)
+		(stroke
+			(width 0)
+			(type default)
+		)
+	)
+	(wire
+		(pts
 			(xy 247.65 119.38) (xy 247.65 127)
 		)
@@
 	(wire
 		(pts
+			(xy 114.3 105.41) (xy 106.68 105.41)
+		)
+		(stroke
+			(width 0)
+			(type default)
+		)
+	)
+	(wire
+		(pts
 			(xy 39.37 93.98) (xy 45.72 93.98)
 		)
@@
 	(wire
 		(pts
+			(xy 113.03 97.79) (xy 113.03 93.98)
+		)
+		(stroke
+			(width 0)
+			(type default)
+		)
+	)
+	(wire
+		(pts
 			(xy 121.92 82.55) (xy 124.46 82.55)
 		)
@@
 	(wire
 		(pts
+			(xy 114.3 102.87) (xy 114.3 105.41)
+		)
+		(stroke
+			(width 0)
+			(type default)
+		)
+	)
+	(wire
+		(pts
 			(xy 137.16 68.58) (xy 137.16 69.85)
 		)
@@
 	(wire
 		(pts
+			(xy 114.3 101.6) (xy 106.68 101.6)
+		)
+		(stroke
+			(width 0)
+			(type default)
+		)
+	)
+	(wire
+		(pts
 			(xy 214.63 107.95) (xy 219.71 107.95)
 		)
@@
 		)
 	)
-	(text "0.95$"
+	(text "1.8$"
 		(exclude_from_sim no)
 		(at 79.756 56.896 0)
@@
 		)
 	)
-	(text "Charger 3"
+	(text "Charger 2\n"
 		(exclude_from_sim no)
 		(at 221.742 55.118 0)
@@
 		)
 	)
-	(text "Charger 2"
+	(text "Charger 3"
 		(exclude_from_sim no)
 		(at 133.35 54.864 0)
@@
 		(dnp no)
 		(fields_autoplaced yes)
-		(property "Reference" "J1"
+		(property "Reference" "STAT3"
 			(at 211.455 119.38 0)
 			(effects
@@
 			(project ""
 				(path "/abe2d707-f40d-456a-8d07-9815f6d9031d"
-					(reference "J1")
+					(reference "STAT3")
 					(unit 1)
 				)
@@
 	(symbol
 		(lib_id "Connector:Conn_01x03_Pin")
-		(at 109.22 100.33 0)
+		(at 111.76 100.33 180)
 		(unit 1)
 		(exclude_from_sim no)
@@
 		(dnp no)
 		(property "Reference" "STAT2"
-			(at 108.458 93.472 0)
+			(at 112.522 107.188 0)
 			(effects
 				(font
@@
 		)
 		(property "Value" "STAT"
-			(at 109.22 96.012 0)
+			(at 111.76 104.648 0)
 			(effects
 				(font
@@
 		)
 		(property "Footprint" "Connector_PinSocket_2.54mm:PinSocket_1x03_P2.54mm_Vertical"
-			(at 109.22 100.33 0)
+			(at 111.76 100.33 0)
 			(effects
 				(font
@@
 		)
 		(property "Datasheet" "~"
-			(at 109.22 100.33 0)
+			(at 111.76 100.33 0)
 			(effects
 				(font
@@
 		)
 		(property "Description" "Generic connector, single row, 01x03, script generated"
-			(at 109.22 100.33 0)
+			(at 111.76 100.33 0)
 			(effects
 				(font
@@
 					(unit 1)
 				)
+			)
+		)
+	)
+	(symbol
+		(lib_id "Connector:TestPoint")
+		(at 59.69 185.42 180)
+		(unit 1)
+		(exclude_from_sim no)
+		(in_bom yes)
+		(on_board yes)
+		(dnp no)
+		(property "Reference" "GND1"
+			(at 59.055 187.96 0)
+			(effects
+				(font
+					(size 1.27 1.27)
+				)
+				(justify left)
+			)
+		)
+		(property "Value" "GND"
+			(at 70.612 190.246 0)
+			(effects
+				(font
+					(size 1.27 1.27)
+				)
+				(justify left)
+			)
+		)
+		(property "Footprint" "TestPoint:TestPoint_Pad_D1.5mm"
+			(at 54.61 185.42 0)
+			(effects
+				(font
+					(size 1.27 1.27)
+				)
+				(hide yes)
+			)
+		)
+		(property "Datasheet" "~"
+			(at 54.61 185.42 0)
+			(effects
+				(font
+					(size 1.27 1.27)
+				)
+				(hide yes)
+			)
+		)
+		(property "Description" ""
+			(at 59.69 185.42 0)
+			(effects
+				(font
+					(size 1.27 1.27)
+				)
+				(hide yes)
+			)
+		)
+		(pin "1"
+		)
+		(instances
+			(project "Li-po_chargers_tester"
+				(path "/abe2d707-f40d-456a-8d07-9815f6d9031d"
+					(reference "GND1")
+					(unit 1)
+				)
